File: scsc/usb-100basefx.brd (EAGLE design)
At the start: 44 x 44 mm, 55 parts, among them IC1 LD33, IC2 93LC66SN, U1 AX88772B, U2 AFBR-5803Z, Y1 25MHz

Commit message: rc: update
Routing:
- net TD_DN: track 49.9 -> 49.1 mm
- net TD_DP: track 49.3 -> 48.5 mm
Changed lines of the file:
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@@
 <contactref element="U2" pad="8"/>
 <contactref element="U1" pad="12"/>
-<via x="29.0576" y="22.5552" extent="1-16" drill="0.508"/>
+<via x="27.6352" y="19.9136" extent="1-16" drill="0.508"/>
 <wire x1="29.464" y1="32.3088" x2="29.464" y2="22.9616" width="0.2032" layer="1"/>
-<wire x1="29.0576" y1="22.5552" x2="29.464" y2="22.9616" width="0.2032" layer="1"/>
+<wire x1="29.464" y1="22.9616" x2="28.0416" y2="21.5392" width="0.2032" layer="1"/>
+<wire x1="28.0416" y1="21.5392" x2="28.0416" y2="20.32" width="0.2032" layer="1"/>
+<wire x1="27.6352" y1="19.9136" x2="28.0416" y2="20.32" width="0.2032" layer="1"/>
 <wire x1="9.7908" y1="9.7536" x2="11.176" y2="9.7536" width="0.4064" layer="1"/>
 <via x="11.176" y="9.7536" extent="1-16" drill="0.508"/>
@@
 <wire x1="16.5598" y1="10.2626" x2="16.5598" y2="10.2616" width="0.4064" layer="1"/>
 <wire x1="11.176" y1="9.7536" x2="11.176" y2="8.5716" width="0.4064" layer="1"/>
-<wire x1="29.0576" y1="22.5552" x2="29.464" y2="22.9616" width="0.2032" layer="16"/>
-<wire x1="29.464" y1="22.9616" x2="29.464" y2="23.7744" width="0.2032" layer="16"/>
-<wire x1="29.464" y1="23.7744" x2="29.0576" y2="24.1808" width="0.2032" layer="16"/>
-<wire x1="29.0576" y1="24.1808" x2="28.448" y2="24.1808" width="0.2032" layer="16"/>
-<wire x1="28.448" y1="24.1808" x2="25.8064" y2="21.5392" width="0.2032" layer="16"/>
-<wire x1="25.8064" y1="21.5392" x2="25.8064" y2="13.8176" width="0.2032" layer="16"/>
-<wire x1="25.8064" y1="13.8176" x2="23.368" y2="11.3792" width="0.2032" layer="16"/>
-<wire x1="23.368" y1="11.3792" x2="14.8336" y2="11.3792" width="0.2032" layer="16"/>
+<wire x1="27.6352" y1="19.9136" x2="28.0416" y2="20.32" width="0.2032" layer="16"/>
+<wire x1="28.0416" y1="20.32" x2="28.0416" y2="21.1328" width="0.2032" layer="16"/>
+<wire x1="28.0416" y1="21.1328" x2="27.6352" y2="21.5392" width="0.2032" layer="16"/>
+<wire x1="27.6352" y1="21.5392" x2="27.0256" y2="21.5392" width="0.2032" layer="16"/>
+<wire x1="27.0256" y1="21.5392" x2="24.384" y2="18.8976" width="0.2032" layer="16"/>
+<wire x1="24.384" y1="18.8976" x2="24.384" y2="13.8176" width="0.2032" layer="16"/>
+<wire x1="24.384" y1="13.8176" x2="21.9456" y2="11.3792" width="0.2032" layer="16"/>
+<wire x1="21.9456" y1="11.3792" x2="14.8336" y2="11.3792" width="0.2032" layer="16"/>
 <wire x1="14.8336" y1="11.3792" x2="13.8176" y2="10.3632" width="0.2032" layer="16"/>
 <wire x1="13.8176" y1="10.3632" x2="11.5824" y2="10.3632" width="0.2032" layer="16"/>
@@
 <contactref element="U2" pad="7"/>
 <contactref element="U1" pad="13"/>
-<via x="30.2768" y="22.5552" extent="1-16" drill="0.508"/>
-<wire x1="29.8704" y1="32.3088" x2="29.8704" y2="22.9616" width="0.2032" layer="1"/>
-<wire x1="30.2768" y1="22.5552" x2="29.8704" y2="22.9616" width="0.2032" layer="1"/>
+<via x="28.8544" y="19.9136" extent="1-16" drill="0.508"/>
+<wire x1="29.8704" y1="32.3088" x2="29.8704" y2="22.7584" width="0.2032" layer="1"/>
+<wire x1="29.8704" y1="22.7584" x2="28.448" y2="21.336" width="0.2032" layer="1"/>
+<wire x1="28.448" y1="21.336" x2="28.448" y2="20.32" width="0.2032" layer="1"/>
+<wire x1="28.8544" y1="19.9136" x2="28.448" y2="20.32" width="0.2032" layer="1"/>
 <wire x1="9.7908" y1="11.176" x2="11.176" y2="11.176" width="0.4064" layer="1"/>
 <via x="11.176" y="11.176" extent="1-16" drill="0.508"/>
@@
 <wire x1="16.5598" y1="12.699" x2="16.5598" y2="12.8016" width="0.4064" layer="1"/>
 <wire x1="11.176" y1="11.176" x2="11.176" y2="12.358" width="0.4064" layer="1"/>
-<wire x1="30.2768" y1="22.5552" x2="29.8704" y2="22.9616" width="0.2032" layer="16"/>
-<wire x1="29.8704" y1="22.9616" x2="29.8704" y2="23.9776" width="0.2032" layer="16"/>
-<wire x1="29.8704" y1="23.9776" x2="29.2608" y2="24.5872" width="0.2032" layer="16"/>
-<wire x1="29.2608" y1="24.5872" x2="28.2448" y2="24.5872" width="0.2032" layer="16"/>
-<wire x1="28.2448" y1="24.5872" x2="25.4" y2="21.7424" width="0.2032" layer="16"/>
-<wire x1="25.4" y1="21.7424" x2="25.4" y2="14.0208" width="0.2032" layer="16"/>
-<wire x1="25.4" y1="14.0208" x2="23.1648" y2="11.7856" width="0.2032" layer="16"/>
-<wire x1="23.1648" y1="11.7856" x2="14.6304" y2="11.7856" width="0.2032" layer="16"/>
+<wire x1="28.8544" y1="19.9136" x2="28.448" y2="20.32" width="0.2032" layer="16"/>
+<wire x1="28.448" y1="20.32" x2="28.448" y2="21.336" width="0.2032" layer="16"/>
+<wire x1="28.448" y1="21.336" x2="27.8384" y2="21.9456" width="0.2032" layer="16"/>
+<wire x1="27.8384" y1="21.9456" x2="26.8224" y2="21.9456" width="0.2032" layer="16"/>
+<wire x1="26.8224" y1="21.9456" x2="23.9776" y2="19.1008" width="0.2032" layer="16"/>
+<wire x1="23.9776" y1="19.1008" x2="23.9776" y2="14.0208" width="0.2032" layer="16"/>
+<wire x1="23.9776" y1="14.0208" x2="21.7424" y2="11.7856" width="0.2032" layer="16"/>
+<wire x1="21.7424" y1="11.7856" x2="14.6304" y2="11.7856" width="0.2032" layer="16"/>
 <wire x1="14.6304" y1="11.7856" x2="13.6144" y2="10.7696" width="0.2032" layer="16"/>
 <wire x1="13.6144" y1="10.7696" x2="11.5824" y2="10.7696" width="0.2032" layer="16"/>
@@
 </signal>
 </signals>
-<errors>
-</errors>
 </board>
 </drawing>

Commit message: hw: change some values
Parts:
- C1, C2: value 1u -> 10u
- C7, C8: value 18p -> 33p
Changed lines of the file:
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@@
 </autorouter>
 <elements>
-<element name="C1" library="rcl" package="C0603" value="1u" x="12.8016" y="19.5072" rot="R90"/>
+<element name="C1" library="rcl" package="C0603" value="10u" x="12.8016" y="19.5072" rot="R90"/>
 <element name="R1" library="rcl" package="R0603" value="130" x="8.9408" y="9.7536"/>
 <element name="LED1" library="led" package="CHIPLED_0805" value="" x="41.4528" y="33.7312" rot="R180"/>
@@
 <element name="U2" library="balto" package="AFBR-5803Z" value="AFBR-5803Z" x="33.3248" y="17.8816" locked="yes"/>
 <element name="BOX1" library="hammond" package="1551R" value="HAMMOND-BOX-R" x="0" y="0"/>
-<element name="C2" library="rcl" package="C0603" value="1u" x="12.8016" y="15.24" rot="R270"/>
+<element name="C2" library="rcl" package="C0603" value="10u" x="12.8016" y="15.24" rot="R270"/>
 <element name="R2" library="rcl" package="R0603" value="82" x="11.176" y="7.7216" rot="R270"/>
 <element name="R3" library="rcl" package="R0603" value="82" x="11.176" y="13.208" rot="R90"/>
@@
 <element name="R14" library="rcl" package="R0603" value="22" x="38.2016" y="21.336" rot="MR0"/>
 <element name="Y1" library="SparkFun-FreqCtrl" package="CRYSTAL-SMD-5X3" value="25MHz" x="14.8336" y="32.9184" rot="R180"/>
-<element name="C7" library="rcl" package="C0603" value="18p" x="14.8336" y="35.3568" rot="R180"/>
-<element name="C8" library="rcl" package="C0603" value="18p" x="12.5984" y="29.464" rot="R270"/>
+<element name="C7" library="rcl" package="C0603" value="33p" x="14.8336" y="35.3568" rot="R180"/>
+<element name="C8" library="rcl" package="C0603" value="33p" x="12.5984" y="29.464" rot="R270"/>
 <element name="R15" library="rcl" package="R0603" value="1M" x="19.304" y="32.512" rot="R270"/>
 <element name="LED2" library="led" package="CHIPLED_0805" value="" x="39.8272" y="33.7312" rot="R180"/>
