File: scsc/usb-100basefx.sch (EAGLE design)
At the start: 59 parts, among them IC1 LD33, IC2 93LC66SN, U1 AX88772B, U2 AFBR-5803Z, Y1 25MHz

Commit message: hw: redone
Parts:
- removed LED3, LED4: (no value), led:LEDCHIPLED_0805
- removed R18, R19: 330, rcl:R-EU_R0603
Connections:
- removed net LED3: R18.2, U1.MFA1/MDIO
- removed net LED4: R19.2, U1.MFA0/MDC
- removed net N$10: LED4.C, R19.1
- removed net N$8: LED2.C, R17.1
- removed net N$9: LED3.C, R18.1
- new net N$6: LED1.A, R16.2
- net LED1: now also LED1.C; no longer R16.2
- net LED2: now also LED2.C; no longer R17.2
- net N$7: now also LED2.A, R17.2; no longer LED1.C, R16.1
- net VCC: now also R16.1, R17.1; no longer LED1.A, LED2.A, LED3.A, LED4.A
Other:
- moved on the sheet: LED1, LED2, R16, R17
Changed lines of the file:
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@@
 <?xml version="1.0" encoding="utf-8"?>
 <!DOCTYPE eagle SYSTEM "eagle.dtd">
-<eagle version="6.3">
+<eagle version="6.4">
 <drawing>
 <settings>
@@
 <part name="R15" library="rcl" deviceset="R-EU_" device="R0603" value="1M"/>
 <part name="LED2" library="led" deviceset="LED" device="CHIPLED_0805"/>
-<part name="LED3" library="led" deviceset="LED" device="CHIPLED_0805"/>
-<part name="LED4" library="led" deviceset="LED" device="CHIPLED_0805"/>
 <part name="R16" library="rcl" deviceset="R-EU_" device="R0603" value="330"/>
 <part name="R17" library="rcl" deviceset="R-EU_" device="R0603" value="330"/>
-<part name="R18" library="rcl" deviceset="R-EU_" device="R0603" value="330"/>
-<part name="R19" library="rcl" deviceset="R-EU_" device="R0603" value="330"/>
 <part name="P+7" library="supply1" deviceset="VCC" device=""/>
 <part name="FRAME2" library="frames" deviceset="DINA4_L" device=""/>
@@
 <wire x1="2.54" y1="2.54" x2="2.54" y2="45.72" width="0.1524" layer="97"/>
 <wire x1="2.54" y1="177.8" x2="53.34" y2="177.8" width="0.1524" layer="97"/>
-<wire x1="53.34" y1="177.8" x2="53.34" y2="139.7" width="0.1524" layer="97"/>
-<wire x1="53.34" y1="139.7" x2="53.34" y2="137.16" width="0.1524" layer="97"/>
-<wire x1="53.34" y1="137.16" x2="53.34" y2="132.08" width="0.1524" layer="97"/>
+<wire x1="53.34" y1="177.8" x2="53.34" y2="132.08" width="0.1524" layer="97"/>
 <wire x1="53.34" y1="132.08" x2="2.54" y2="132.08" width="0.1524" layer="97"/>
 <wire x1="2.54" y1="132.08" x2="2.54" y2="177.8" width="0.1524" layer="97"/>
-<wire x1="60.96" y1="177.8" x2="109.22" y2="177.8" width="0.1524" layer="97"/>
+<wire x1="55.88" y1="177.8" x2="109.22" y2="177.8" width="0.1524" layer="97"/>
 <wire x1="109.22" y1="177.8" x2="109.22" y2="132.08" width="0.1524" layer="97"/>
 <wire x1="109.22" y1="132.08" x2="55.88" y2="132.08" width="0.1524" layer="97"/>
 <wire x1="55.88" y1="132.08" x2="55.88" y2="177.8" width="0.1524" layer="97"/>
-<wire x1="55.88" y1="177.8" x2="60.96" y2="177.8" width="0.1524" layer="97"/>
 <wire x1="83.82" y1="35.56" x2="160.02" y2="35.56" width="0.1524" layer="97"/>
 <wire x1="160.02" y1="35.56" x2="160.02" y2="2.54" width="0.1524" layer="97"/>
@@
 <attribute name="VALUE" x="17.78" y="106.68" size="1.778" layer="96"/>
 </instance>
-<instance part="LED1" gate="G$1" x="68.58" y="162.56"/>
+<instance part="LED1" gate="G$1" x="78.74" y="149.86"/>
 <instance part="GND1" gate="1" x="86.36" y="58.42"/>
 <instance part="P+1" gate="VCC" x="86.36" y="81.28"/>
@@
 <attribute name="VALUE" x="243.84" y="119.38" size="1.778" layer="96"/>
 </instance>
-<instance part="LED2" gate="G$1" x="78.74" y="162.56"/>
-<instance part="LED3" gate="G$1" x="88.9" y="162.56"/>
-<instance part="LED4" gate="G$1" x="99.06" y="162.56"/>
-<instance part="R16" gate="G$1" x="68.58" y="149.86" smashed="yes" rot="R270">
-<attribute name="NAME" x="71.12" y="149.86" size="1.778" layer="95"/>
-<attribute name="VALUE" x="71.12" y="147.32" size="1.778" layer="96"/>
-</instance>
-<instance part="R17" gate="G$1" x="78.74" y="149.86" smashed="yes" rot="R270">
-<attribute name="NAME" x="81.28" y="149.86" size="1.778" layer="95"/>
-<attribute name="VALUE" x="81.28" y="147.32" size="1.778" layer="96"/>
-</instance>
-<instance part="R18" gate="G$1" x="88.9" y="149.86" smashed="yes" rot="R270">
-<attribute name="NAME" x="91.44" y="149.86" size="1.778" layer="95"/>
-<attribute name="VALUE" x="91.44" y="147.32" size="1.778" layer="96"/>
-</instance>
-<instance part="R19" gate="G$1" x="99.06" y="149.86" smashed="yes" rot="R270">
-<attribute name="NAME" x="101.6" y="149.86" size="1.778" layer="95"/>
-<attribute name="VALUE" x="101.6" y="147.32" size="1.778" layer="96"/>
+<instance part="LED2" gate="G$1" x="88.9" y="149.86"/>
+<instance part="R16" gate="G$1" x="78.74" y="160.02" smashed="yes" rot="R270">
+<attribute name="NAME" x="81.28" y="160.02" size="1.778" layer="95"/>
+<attribute name="VALUE" x="81.28" y="157.48" size="1.778" layer="96"/>
+</instance>
+<instance part="R17" gate="G$1" x="88.9" y="160.02" smashed="yes" rot="R270">
+<attribute name="NAME" x="91.44" y="160.02" size="1.778" layer="95"/>
+<attribute name="VALUE" x="91.44" y="157.48" size="1.778" layer="96"/>
 </instance>
 <instance part="P+7" gate="VCC" x="83.82" y="172.72"/>
@@
 <segment>
 <pinref part="P+7" gate="VCC" pin="VCC"/>
-<wire x1="68.58" y1="167.64" x2="78.74" y2="167.64" width="0.1524" layer="91"/>
 <wire x1="78.74" y1="167.64" x2="83.82" y2="167.64" width="0.1524" layer="91"/>
 <wire x1="83.82" y1="167.64" x2="83.82" y2="170.18" width="0.1524" layer="91"/>
+<pinref part="R16" gate="G$1" pin="1"/>
+<wire x1="78.74" y1="167.64" x2="78.74" y2="165.1" width="0.1524" layer="91"/>
+<pinref part="R17" gate="G$1" pin="1"/>
 <wire x1="83.82" y1="167.64" x2="88.9" y2="167.64" width="0.1524" layer="91"/>
+<wire x1="88.9" y1="167.64" x2="88.9" y2="165.1" width="0.1524" layer="91"/>
 <junction x="83.82" y="167.64"/>
-<wire x1="88.9" y1="167.64" x2="99.06" y2="167.64" width="0.1524" layer="91"/>
-<pinref part="LED1" gate="G$1" pin="A"/>
-<wire x1="68.58" y1="165.1" x2="68.58" y2="167.64" width="0.1524" layer="91"/>
-<pinref part="LED2" gate="G$1" pin="A"/>
-<wire x1="78.74" y1="165.1" x2="78.74" y2="167.64" width="0.1524" layer="91"/>
-<junction x="78.74" y="167.64"/>
-<pinref part="LED3" gate="G$1" pin="A"/>
-<wire x1="88.9" y1="165.1" x2="88.9" y2="167.64" width="0.1524" layer="91"/>
-<junction x="88.9" y="167.64"/>
-<pinref part="LED4" gate="G$1" pin="A"/>
-<wire x1="99.06" y1="165.1" x2="99.06" y2="167.64" width="0.1524" layer="91"/>
 </segment>
 <segment>
@@
 <net name="LED1" class="0">
 <segment>
-<wire x1="68.58" y1="142.24" x2="58.42" y2="142.24" width="0.1524" layer="91"/>
-<label x="58.42" y="142.24" size="1.778" layer="95"/>
-<pinref part="R16" gate="G$1" pin="2"/>
-<wire x1="68.58" y1="144.78" x2="68.58" y2="142.24" width="0.1524" layer="91"/>
+<wire x1="78.74" y1="142.24" x2="68.58" y2="142.24" width="0.1524" layer="91"/>
+<label x="68.58" y="142.24" size="1.778" layer="95"/>
+<pinref part="LED1" gate="G$1" pin="C"/>
+<wire x1="78.74" y1="142.24" x2="78.74" y2="144.78" width="0.1524" layer="91"/>
 </segment>
 <segment>
@@
 <net name="LED2" class="0">
 <segment>
-<wire x1="78.74" y1="139.7" x2="58.42" y2="139.7" width="0.1524" layer="91"/>
-<label x="58.42" y="139.7" size="1.778" layer="95"/>
-<pinref part="R17" gate="G$1" pin="2"/>
-<wire x1="78.74" y1="139.7" x2="78.74" y2="144.78" width="0.1524" layer="91"/>
+<wire x1="88.9" y1="139.7" x2="68.58" y2="139.7" width="0.1524" layer="91"/>
+<label x="68.58" y="139.7" size="1.778" layer="95"/>
+<pinref part="LED2" gate="G$1" pin="C"/>
+<wire x1="88.9" y1="139.7" x2="88.9" y2="144.78" width="0.1524" layer="91"/>
 </segment>
 <segment>
@@
 <wire x1="220.98" y1="83.82" x2="233.68" y2="83.82" width="0.1524" layer="91"/>
 <label x="233.68" y="83.82" size="1.778" layer="95" rot="MR0"/>
-</segment>
-</net>
-<net name="LED3" class="0">
-<segment>
-<wire x1="88.9" y1="137.16" x2="58.42" y2="137.16" width="0.1524" layer="91"/>
-<label x="58.42" y="137.16" size="1.778" layer="95"/>
-<pinref part="R18" gate="G$1" pin="2"/>
-<wire x1="88.9" y1="137.16" x2="88.9" y2="144.78" width="0.1524" layer="91"/>
-</segment>
-<segment>
-<pinref part="U1" gate="G$1" pin="MFA1/MDIO"/>
-<wire x1="220.98" y1="81.28" x2="233.68" y2="81.28" width="0.1524" layer="91"/>
-<label x="233.68" y="81.28" size="1.778" layer="95" rot="MR0"/>
-</segment>
-</net>
-<net name="LED4" class="0">
-<segment>
-<wire x1="99.06" y1="134.62" x2="58.42" y2="134.62" width="0.1524" layer="91"/>
-<label x="58.42" y="134.62" size="1.778" layer="95"/>
-<pinref part="R19" gate="G$1" pin="2"/>
-<wire x1="99.06" y1="134.62" x2="99.06" y2="144.78" width="0.1524" layer="91"/>
-</segment>
-<segment>
-<pinref part="U1" gate="G$1" pin="MFA0/MDC"/>
-<wire x1="220.98" y1="78.74" x2="233.68" y2="78.74" width="0.1524" layer="91"/>
-<label x="233.68" y="78.74" size="1.778" layer="95" rot="MR0"/>
 </segment>
 </net>
@@
 </segment>
 </net>
-<net name="N$7" class="0">
-<segment>
-<pinref part="LED1" gate="G$1" pin="C"/>
-<pinref part="R16" gate="G$1" pin="1"/>
-<wire x1="68.58" y1="154.94" x2="68.58" y2="157.48" width="0.1524" layer="91"/>
-</segment>
-</net>
-<net name="N$8" class="0">
-<segment>
-<pinref part="LED2" gate="G$1" pin="C"/>
-<pinref part="R17" gate="G$1" pin="1"/>
-<wire x1="78.74" y1="154.94" x2="78.74" y2="157.48" width="0.1524" layer="91"/>
-</segment>
-</net>
-<net name="N$9" class="0">
-<segment>
-<pinref part="LED3" gate="G$1" pin="C"/>
-<pinref part="R18" gate="G$1" pin="1"/>
-<wire x1="88.9" y1="154.94" x2="88.9" y2="157.48" width="0.1524" layer="91"/>
-</segment>
-</net>
-<net name="N$10" class="0">
-<segment>
-<pinref part="LED4" gate="G$1" pin="C"/>
-<pinref part="R19" gate="G$1" pin="1"/>
-<wire x1="99.06" y1="154.94" x2="99.06" y2="157.48" width="0.1524" layer="91"/>
-</segment>
-</net>
 <net name="RD_DN" class="0">
 <segment>
@@
 </segment>
 </net>
+<net name="N$6" class="0">
+<segment>
+<pinref part="LED1" gate="G$1" pin="A"/>
+<pinref part="R16" gate="G$1" pin="2"/>
+<wire x1="78.74" y1="152.4" x2="78.74" y2="154.94" width="0.1524" layer="91"/>
+</segment>
+</net>
+<net name="N$7" class="0">
+<segment>
+<pinref part="LED2" gate="G$1" pin="A"/>
+<pinref part="R17" gate="G$1" pin="2"/>
+<wire x1="88.9" y1="152.4" x2="88.9" y2="154.94" width="0.1524" layer="91"/>
+</segment>
+</net>

Commit message: hw: change some values
Parts:
- C1, C2: value 1u -> 10u
- C7, C8: value 18p -> 33p
Changed lines of the file:
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@@
 </classes>
 <parts>
-<part name="C1" library="rcl" deviceset="C-EU" device="C0603" value="1u"/>
+<part name="C1" library="rcl" deviceset="C-EU" device="C0603" value="10u"/>
 <part name="R1" library="rcl" deviceset="R-EU_" device="R0603" value="130"/>
 <part name="LED1" library="led" deviceset="LED" device="CHIPLED_0805"/>
@@
 <part name="U2" library="balto" deviceset="AFBR-5803Z" device=""/>
 <part name="BOX1" library="hammond" deviceset="HAMMOND-BOX" device="-R"/>
-<part name="C2" library="rcl" deviceset="C-EU" device="C0603" value="1u"/>
+<part name="C2" library="rcl" deviceset="C-EU" device="C0603" value="10u"/>
 <part name="P+2" library="supply1" deviceset="VCC" device=""/>
 <part name="GND2" library="supply1" deviceset="GND" device=""/>
@@
 <part name="GND12" library="supply1" deviceset="GND" device=""/>
 <part name="Y1" library="SparkFun-FreqCtrl" deviceset="CRYSTAL" device="5X3" value="25MHz"/>
-<part name="C7" library="rcl" deviceset="C-EU" device="C0603" value="18p"/>
-<part name="C8" library="rcl" deviceset="C-EU" device="C0603" value="18p"/>
+<part name="C7" library="rcl" deviceset="C-EU" device="C0603" value="33p"/>
+<part name="C8" library="rcl" deviceset="C-EU" device="C0603" value="33p"/>
 <part name="GND13" library="supply1" deviceset="GND" device=""/>
 <part name="GND14" library="supply1" deviceset="GND" device=""/>
